Commit message: add imu link,  modif on lidar and start p3d config

File: tekbot_description/urdf/tekbot.urdf (robot description, URDF)
Before this commit: robot tekbot, 4 links, 3 joints
Links:
- removed link dummy_link
- added link imu_link; visual box size=0.02 0.02 0.02
- link lidar_link: geometry visual cylinder length=0.1 radius=0.03
Joints:
- removed joint dummy_joint
- added joint imu_joint: type fixed, parent base_link, child imu_link, origin xyz=0 0 0.01 rpy=0 0 0
- joint lidar_joint: origin xyz=0.1 0.0 0.05 rpy=0 0 0 -> xyz=0.1 0.0 0.075 rpy=0 0 0
