Commit message: add ekf loc and teleop

File: tekbot_description/urdf/cylinder.urdf.xacro (robot description, xacro)
@@ -5,5 +5,10 @@
             <origin xyz="0 0 0" rpy="${pi/2} 0 0" />
             <mass value="${m}"/>
-            <inertia ixx="${(m/12) * (3*r*r + h*h)}" ixy = "0" ixz = "0" iyy="${(m/12) * (3*r*r + h*h)}" iyz = "0" izz="${(m/2) * (r*r)}"/>
+            <inertia ixx="${(m/12) * (3*r*r + h*h)}"
+                     ixy = "0"
+                     ixz = "0"
+                     iyy="${(m/12) * (3*r*r + h*h)}"
+                     iyz = "0"
+                     izz="${(m/2) * (r*r)}"/>
         </inertial>
     </xacro:macro>
